Commit message: feat: Add initial WPF TeachPendant main window and associated build artifacts.

File: TeachPendant_WPF/Assets/robot.urdf (robot description, URDF)
Before this commit: robot robot_6_dof, 7 links, 6 joints
Links:
- link base_link: geometry visual cylinder length=0.05 radius=0.10; visual cylinder length=0.05 radius=0.15
- link link_1: geometry visual cylinder length=0.12 radius=0.085
- link link_2: geometry visual cylinder length=0.06 radius=0.07; visual cylinder length=0.35 radius=0.055
- link link_3: geometry visual cylinder length=0.05 radius=0.06; visual cylinder length=0.26 radius=0.045
- link link_4: geometry visual cylinder length=0.08 radius=0.04
- link link_5: geometry visual cylinder length=0.07 radius=0.035
- link link_6: geometry visual box size=0.05 0.05 0.015; visual cylinder length=0.015 radius=0.03
Joints:
- joint joint_1: limit (none) -> lower=-2.967 upper=2.967
- joint joint_2: limit (none) -> lower=-2.094 upper=2.094; origin xyz=0 0 0.1 rpy=-1.57079632679 0 0 -> xyz=0 0 0.12 rpy=-1.5707963 0 0
- joint joint_3: limit (none) -> lower=-2.967 upper=2.967; origin xyz=0.4 0 0 rpy=0 0 0 -> xyz=0.35 0 0 rpy=0 0 0
- joint joint_4: limit (none) -> lower=-3.14159 upper=3.14159; origin xyz=0.3 0 0 rpy=0 0 0 -> xyz=0.26 0 0 rpy=0 0 0
- joint joint_5: limit (none) -> lower=-2.094 upper=2.094; origin xyz=0 0.05 0 rpy=1.57079632679 0 0 -> xyz=0 0.04 0 rpy=1.5707963 0 0
- joint joint_6: limit (none) -> lower=-6.283 upper=6.283; origin xyz=0 0 0.08 rpy=-1.57079632679 0 0 -> xyz=0 0 0.07 rpy=-1.5707963 0 0
