Commit message: New connected software backend -g

File: src/robot_description/urdf/custom_6axis_test.urdf.xacro (robot description, xacro)
@@ -1,47 +1,64 @@
 <?xml version="1.0"?>
-<robot xmlns:xacro="http://www.ros.org/wiki/xacro" name="robot_arm">
+<robot xmlns:xacro="http://www.ros.org/wiki/xacro" name="industrial_6dof">
   <!-- Materials -->
-  <material name="orange">
-    <color rgba="1.0 0.5 0.0 1.0"/>
+  <material name="industrial_orange">
+    <color rgba="1.0 0.4 0.0 1.0"/>
   </material>
-  <material name="grey">
-    <color rgba="0.2 0.2 0.2 1.0"/>
+  <material name="industrial_dark">
+    <color rgba="0.2 0.2 0.22 1.0"/>
   </material>
-  <!-- Base Link -->
+  <material name="industrial_silver">
+    <color rgba="0.75 0.75 0.75 1.0"/>
+  </material>
+  <!-- ======================== CONSTANTS ======================== -->
+  <!-- pi is natively built into newer xacro versions -->
+  <!-- ======================== LINKS & JOINTS ======================== -->
+  <!-- Dummy root link to prevent KDL & Gazebo root inertia errors -->
+  <link name="world"/>
+  <joint name="fixed_base_joint" type="fixed">
+    <parent link="world"/>
+    <child link="base_link"/>
+    <origin xyz="0 0 0" rpy="0 0 0"/>
+  </joint>
+  <!-- Base Link (Pedestal) -->
   <link name="base_link">
     <visual>
       <geometry>
-        <cylinder length="0.1" radius="0.15"/>
-      </geometry>
-      <material name="grey"/>
-    </visual>
-    <collision>
-      <geometry>
-        <cylinder length="0.1" radius="0.15"/>
-      </geometry>
-    </collision>
-    <inertial>
-      <mass value="5.0"/>
-      <inertia ixx="0.1" ixy="0.0" ixz="0.0" iyy="0.1" iyz="0.0" izz="0.1"/>
-    </inertial>
-  </link>
-  <!-- Link 1 -->
+        <cylinder length="0.15" radius="0.18"/>
+      </geometry>
+      <origin xyz="0 0 0.075" rpy="0 0 0"/>
+      <material name="industrial_dark"/>
+    </visual>
+    <collision>
+      <geometry>
+        <cylinder length="0.15" radius="0.18"/>
+      </geometry>
+      <origin xyz="0 0 0.075" rpy="0 0 0"/>
+    </collision>
+    <inertial>
+      <mass value="15.0"/>
+      <origin xyz="0 0 0.075" rpy="0 0 0"/>
+      <inertia ixx="0.2" ixy="0.0" ixz="0.0" iyy="0.2" iyz="0.0" izz="0.4"/>
+    </inertial>
+  </link>
+  <!-- Link 1 (Shoulder Pan) -->
   <link name="link_1">
     <visual>
       <geometry>
-        <cylinder length="0.4" radius="0.1"/>
-      </geometry>
-      <origin xyz="0 0 0.2" rpy="0 0 0"/>
-      <material name="orange"/>
-    </visual>
-    <collision>
-      <geometry>
-        <cylinder length="0.4" radius="0.1"/>
-      </geometry>
-      <origin xyz="0 0 0.2" rpy="0 0 0"/>
-    </collision>
-    <inertial>
-      <mass value="3.0"/>
-      <inertia ixx="0.1" ixy="0.0" ixz="0.0" iyy="0.1" iyz="0.0" izz="0.1"/>
+        <cylinder length="0.25" radius="0.14"/>
+      </geometry>
+      <origin xyz="0 0 0.125" rpy="0 0 0"/>
+      <material name="industrial_orange"/>
+    </visual>
+    <collision>
+      <geometry>
+        <cylinder length="0.25" radius="0.14"/>
+      </geometry>
+      <origin xyz="0 0 0.125" rpy="0 0 0"/>
+    </collision>
+    <inertial>
+      <mass value="12.0"/>
+      <origin xyz="0 0 0.125" rpy="0 0 0"/>
+      <inertia ixx="0.15" ixy="0.0" ixz="0.0" iyy="0.15" iyz="0.0" izz="0.1"/>
     </inertial>
   </link>
@@ -49,27 +66,37 @@
     <parent link="base_link"/>
     <child link="link_1"/>
-    <origin xyz="0 0 0.05" rpy="0 0 0"/>
-    <axis xyz="0 0 1"/>
-    <limit lower="-2.96" upper="2.96" effort="100" velocity="1.0"/>
-    <dynamics damping="0.7"/>
-  </joint>
-  <!-- Link 2 -->
+    <origin xyz="0 0 0.15" rpy="0 0 0"/>
+    <axis xyz="0 0 1"/>
+    <limit lower="-2.96" upper="2.96" effort="300" velocity="2.1"/>
+    <dynamics damping="10.0" friction="5.0"/>
+  </joint>
+  <!-- Link 2 (Shoulder Lift / Upper Arm) -->
   <link name="link_2">
     <visual>
-      <geometry>
-        <box size="0.1 0.1 0.5"/>
-      </geometry>
-      <origin xyz="0 0 0.25" rpy="0 0 0"/>
-      <material name="grey"/>
-    </visual>
-    <collision>
-      <geometry>
-        <box size="0.1 0.1 0.5"/>
-      </geometry>
-      <origin xyz="0 0 0.25" rpy="0 0 0"/>
-    </collision>
-    <inertial>
-      <mass value="2.0"/>
-      <inertia ixx="0.05" ixy="0.0" ixz="0.0" iyy="0.05" iyz="0.0" izz="0.05"/>
+      <!-- Main Arm -->
+      <geometry>
+        <cylinder length="0.45" radius="0.09"/>
+      </geometry>
+      <origin xyz="0 0 0.225" rpy="0 0 0"/>
+      <material name="industrial_orange"/>
+    </visual>
+    <visual>
+      <!-- Shoulder Joint Cap -->
+      <geometry>
+        <cylinder length="0.16" radius="0.11"/>
+      </geometry>
+      <origin xyz="0 0 0" rpy="${pi/2} 0 0"/>
+      <material name="industrial_dark"/>
+    </visual>
+    <collision>
+      <geometry>
+        <cylinder length="0.45" radius="0.09"/>
+      </geometry>
+      <origin xyz="0 0 0.225" rpy="0 0 0"/>
+    </collision>
+    <inertial>
+      <mass value="10.0"/>
+      <origin xyz="0 0 0.225" rpy="0 0 0"/>
+      <inertia ixx="0.3" ixy="0.0" ixz="0.0" iyy="0.3" iyz="0.0" izz="0.05"/>
     </inertial>
   </link>
@@ -77,27 +104,37 @@
     <parent link="link_1"/>
     <child link="link_2"/>
-    <origin xyz="0 0 0.4" rpy="0 1.5708 0"/>
-    <axis xyz="0 1 0"/>
-    <limit lower="-2.3" upper="2.3" effort="100" velocity="1.0"/>
-    <dynamics damping="0.7"/>
-  </joint>
-  <!-- Link 3 -->
+    <origin xyz="0 0.05 0.25" rpy="${pi/2} 0 0"/> <!-- Rotated so Link 2 extends outwards -->
+    <axis xyz="0 0 1"/>
+    <limit lower="-2.35" upper="2.35" effort="300" velocity="2.1"/>
+    <dynamics damping="10.0" friction="5.0"/>
+  </joint>
+  <!-- Link 3 (Elbow) -->
   <link name="link_3">
     <visual>
-      <geometry>
-         <cylinder length="0.4" radius="0.08"/>
-      </geometry>
-      <origin xyz="0 0 0.2" rpy="0 0 0"/>
-      <material name="orange"/>
-    </visual>
-    <collision>
-      <geometry>
-        <cylinder length="0.4" radius="0.08"/>
-      </geometry>
-      <origin xyz="0 0 0.2" rpy="0 0 0"/>
-    </collision>
-    <inertial>
-      <mass value="2.0"/>
-      <inertia ixx="0.05" ixy="0.0" ixz="0.0" iyy="0.05" iyz="0.0" izz="0.05"/>
+      <!-- Forearm Base -->
+      <geometry>
+        <cylinder length="0.15" radius="0.08"/>
+      </geometry>
+      <origin xyz="0 0 0.075" rpy="0 0 0"/>
+      <material name="industrial_orange"/>
+    </visual>
+    <visual>
+      <!-- Elbow Joint Cap -->
+      <geometry>
+        <cylinder length="0.14" radius="0.095"/>
+      </geometry>
+      <origin xyz="0 0 0" rpy="${pi/2} 0 0"/>
+      <material name="industrial_dark"/>
+    </visual>
+    <collision>
+      <geometry>
+        <cylinder length="0.15" radius="0.08"/>
+      </geometry>
+      <origin xyz="0 0 0.075" rpy="0 0 0"/>
+    </collision>
+    <inertial>
+      <mass value="8.0"/>
+      <origin xyz="0 0 0.075" rpy="0 0 0"/>
+      <inertia ixx="0.05" ixy="0.0" ixz="0.0" iyy="0.05" iyz="0.0" izz="0.03"/>
     </inertial>
   </link>
@@ -105,27 +142,28 @@
     <parent link="link_2"/>
     <child link="link_3"/>
-    <origin xyz="0 0 0.5" rpy="0 0 0"/>
-    <axis xyz="0 1 0"/>
-    <limit lower="-2.0" upper="2.0" effort="100" velocity="1.0"/>
-    <dynamics damping="0.5"/>
-  </joint>
-  <!-- Link 4 -->
+    <origin xyz="0 0 0.45" rpy="0 0 0"/>
+    <axis xyz="0 0 1"/>
+    <limit lower="-2.61" upper="2.61" effort="150" velocity="2.5"/>
+    <dynamics damping="5.0" friction="2.0"/>
+  </joint>
+  <!-- Link 4 (Forearm Roll) -->
   <link name="link_4">
     <visual>
       <geometry>
-        <cylinder length="0.2" radius="0.06"/>
-      </geometry>
-      <origin xyz="0 0 0.1" rpy="0 0 0"/>
-      <material name="grey"/>
-    </visual>
-    <collision>
-      <geometry>
-        <cylinder length="0.2" radius="0.06"/>
-      </geometry>
-      <origin xyz="0 0 0.1" rpy="0 0 0"/>
-    </collision>
-    <inertial>
-      <mass value="1.0"/>
-      <inertia ixx="0.03" ixy="0.0" ixz="0.0" iyy="0.03" iyz="0.0" izz="0.03"/>
+        <cylinder length="0.35" radius="0.06"/>
+      </geometry>
+      <origin xyz="0 0 0.175" rpy="0 0 0"/>
+      <material name="industrial_silver"/>
+    </visual>
+    <collision>
+      <geometry>
+        <cylinder length="0.35" radius="0.06"/>
+      </geometry>
+      <origin xyz="0 0 0.175" rpy="0 0 0"/>
+    </collision>
+    <inertial>
+      <mass value="5.0"/>
+      <origin xyz="0 0 0.175" rpy="0 0 0"/>
+      <inertia ixx="0.1" ixy="0.0" ixz="0.0" iyy="0.1" iyz="0.0" izz="0.02"/>
     </inertial>
   </link>
@@ -133,27 +171,36 @@
     <parent link="link_3"/>
     <child link="link_4"/>
-    <origin xyz="0 0 0.4" rpy="1.5708 0 0"/>
-    <axis xyz="0 0 1"/>
-    <limit lower="-3.0" upper="3.0" effort="50" velocity="2.0"/>
-    <dynamics damping="0.5"/>
-  </joint>
-  <!-- Link 5 -->
+    <origin xyz="0 -0.05 0.15" rpy="${-pi/2} 0 0"/>
+    <axis xyz="0 0 1"/>
+    <limit lower="-3.14" upper="3.14" effort="100" velocity="3.0"/>
+    <dynamics damping="3.0" friction="1.0"/>
+  </joint>
+  <!-- Link 5 (Wrist Pitch) -->
   <link name="link_5">
     <visual>
       <geometry>
-        <cylinder length="0.15" radius="0.05"/>
-      </geometry>
-      <origin xyz="0 0 0.075" rpy="0 0 0"/>
-      <material name="orange"/>
-    </visual>
-    <collision>
-      <geometry>
-        <cylinder length="0.15" radius="0.05"/>
-      </geometry>
-      <origin xyz="0 0 0.075" rpy="0 0 0"/>
-    </collision>
-    <inertial>
-      <mass value="1.0"/>
-      <inertia ixx="0.02" ixy="0.0" ixz="0.0" iyy="0.02" iyz="0.0" izz="0.02"/>
+        <cylinder length="0.12" radius="0.05"/>
+      </geometry>
+      <origin xyz="0 0 0.06" rpy="0 0 0"/>
+      <material name="industrial_dark"/>
+    </visual>
+    <visual>
+      <!-- Wrist Joint Cap -->
+      <geometry>
+        <cylinder length="0.1" radius="0.06"/>
+      </geometry>
+      <origin xyz="0 0 0" rpy="${pi/2} 0 0"/>
+      <material name="industrial_silver"/>
+    </visual>
+    <collision>
+      <geometry>
+        <cylinder length="0.12" radius="0.05"/>
+      </geometry>
+      <origin xyz="0 0 0.06" rpy="0 0 0"/>
+    </collision>
+    <inertial>
+      <mass value="2.0"/>
+      <origin xyz="0 0 0.06" rpy="0 0 0"/>
+      <inertia ixx="0.01" ixy="0.0" ixz="0.0" iyy="0.01" iyz="0.0" izz="0.01"/>
     </inertial>
   </link>
@@ -161,27 +208,28 @@
     <parent link="link_4"/>
     <child link="link_5"/>
-    <origin xyz="0 0 0.2" rpy="-1.5708 0 0"/>
-    <axis xyz="0 1 0"/>
-    <limit lower="-2.0" upper="2.0" effort="50" velocity="2.0"/>
-    <dynamics damping="0.5"/>
-  </joint>
-  <!-- Link 6 -->
+    <origin xyz="0 0 0.35" rpy="${pi/2} 0 0"/>
+    <axis xyz="0 0 1"/>
+    <limit lower="-2.09" upper="2.09" effort="50" velocity="3.0"/>
+    <dynamics damping="1.0" friction="0.5"/>
+  </joint>
+  <!-- Link 6 (Wrist Roll / Flange) -->
   <link name="link_6">
     <visual>
       <geometry>
-        <cylinder length="0.05" radius="0.04"/>
-      </geometry>
-      <origin xyz="0 0 0.025" rpy="0 0 0"/>
-      <material name="grey"/>
-    </visual>
-    <collision>
-      <geometry>
-        <cylinder length="0.05" radius="0.04"/>
-      </geometry>
-      <origin xyz="0 0 0.025" rpy="0 0 0"/>
+        <cylinder length="0.02" radius="0.045"/>
+      </geometry>
+      <origin xyz="0 0 0.01" rpy="0 0 0"/>
+      <material name="industrial_silver"/>
+    </visual>
+    <collision>
+      <geometry>
+        <cylinder length="0.02" radius="0.045"/>
+      </geometry>
+      <origin xyz="0 0 0.01" rpy="0 0 0"/>
     </collision>
     <inertial>
       <mass value="0.5"/>
-      <inertia ixx="0.01" ixy="0.0" ixz="0.0" iyy="0.01" iyz="0.0" izz="0.01"/>
+      <origin xyz="0 0 0.01" rpy="0 0 0"/>
+      <inertia ixx="0.001" ixy="0.0" ixz="0.0" iyy="0.001" iyz="0.0" izz="0.001"/>
     </inertial>
   </link>
@@ -189,8 +237,8 @@
     <parent link="link_5"/>
     <child link="link_6"/>
-    <origin xyz="0 0 0.15" rpy="1.5708 0 0"/>
-    <axis xyz="0 0 1"/>
-    <limit lower="-6.28" upper="6.28" effort="30" velocity="3.0"/>
-    <dynamics damping="0.1"/>
+    <origin xyz="0 -0.05 0.12" rpy="${-pi/2} 0 0"/>
+    <axis xyz="0 0 1"/>
+    <limit lower="-6.28" upper="6.28" effort="20" velocity="4.0"/>
+    <dynamics damping="0.5" friction="0.1"/>
   </joint>
   <!-- Tool0 -->
@@ -199,10 +247,18 @@
     <parent link="link_6"/>
     <child link="tool0"/>
-    <origin xyz="0 0 0.05" rpy="0 0 0"/>
-  </joint>
-  <!-- ROS 2 Control Tag -->
+    <origin xyz="0 0 0.02" rpy="0 0 0"/>
+  </joint>
+  <!-- ======================== GAZEBO COLORS ======================== -->
+  <gazebo reference="base_link"><material>Gazebo/DarkGrey</material></gazebo>
+  <gazebo reference="link_1"><material>Gazebo/Orange</material></gazebo>
+  <gazebo reference="link_2"><material>Gazebo/Orange</material></gazebo>
+  <gazebo reference="link_3"><material>Gazebo/Orange</material></gazebo>
+  <gazebo reference="link_4"><material>Gazebo/Grey</material></gazebo>
+  <gazebo reference="link_5"><material>Gazebo/DarkGrey</material></gazebo>
+  <gazebo reference="link_6"><material>Gazebo/Grey</material></gazebo>
+  <!-- ======================== ROS 2 CONTROL ======================== -->
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
File: src/robot_description/urdf/robot.urdf.xacro (robot description, xacro)
@@ -29,4 +29,12 @@
     <color rgba="1.0 0.5 0.0 1"/>
   </material>
+  <!-- Dummy root link to satisfy KDL parser & Gazebo -->
+  <link name="world"/>
+  <joint name="fixed_base_joint" type="fixed">
+    <parent link="world"/>
+    <child link="base_link"/>
+    <origin xyz="0 0 0" rpy="0 0 0"/>
+  </joint>
+  <!-- ======================== LINKS & JOINTS ======================== -->
   <!-- ============== BASE LINK ============== -->
   <link name="base_link">
@@ -235,13 +243,18 @@
   </joint>
   <link name="tool0"/>
-  <!-- ============== GAZEBO PLUGINS ============== -->
+  <!-- ============== GAZEBO HARMONIC PLUGINS ============== -->
   <!-- CRITICAL: Remapping maintained -->
   <gazebo>
-    <plugin filename="libgazebo_ros2_control.so" name="gazebo_ros2_control">
-      <robot_sim_type>gazebo_ros2_control/GazeboSystem</robot_sim_type>
-      <parameters>$(find robot_gazebo)/config/gazebo_controllers.yaml</parameters>
-      <ros>
-        <remapping>/joint_states:=/gazebo/joint_states</remapping>
-      </ros>
+    <plugin filename="gz-sim-joint-trajectory-controller-system" name="gz::sim::systems::JointTrajectoryController">
+      <topic>/gazebo/joint_trajectory</topic>
+    </plugin>
+    <plugin filename="gz-sim-joint-state-publisher-system" name="gz::sim::systems::JointStatePublisher">
+      <topic>/gazebo/joint_states</topic>
+      <joint_name>joint_1</joint_name>
+      <joint_name>joint_2</joint_name>
+      <joint_name>joint_3</joint_name>
+      <joint_name>joint_4</joint_name>
+      <joint_name>joint_5</joint_name>
+      <joint_name>joint_6</joint_name>
     </plugin>
   </gazebo>
