Commit message: a

File: RoboForge_WPF/Assets/robot.urdf (robot description, URDF)
Before this commit: robot industrial_6dof, 9 links, 8 joints
Joints:
- joint joint_2: origin xyz=0 0.05 0.25 rpy=${pi/2} 0 0 -> xyz=0 0.05 0.25 rpy=1.5707963267948966 0 0
- joint joint_4: origin xyz=0 -0.05 0.15 rpy=${-pi/2} 0 0 -> xyz=0 -0.05 0.15 rpy=-1.5707963267948966 0 0
- joint joint_5: origin xyz=0 0 0.35 rpy=${pi/2} 0 0 -> xyz=0 0 0.35 rpy=1.5707963267948966 0 0
- joint joint_6: origin xyz=0 -0.05 0.12 rpy=${-pi/2} 0 0 -> xyz=0 -0.05 0.12 rpy=-1.5707963267948966 0 0

File: src/robot_description/urdf/robot.urdf.xacro (robot description, xacro)
@@ -246,8 +246,8 @@
   <!-- CRITICAL: Remapping maintained -->
   <gazebo>
-    <plugin filename="gz-sim-joint-trajectory-controller-system" name="gz::sim::systems::JointTrajectoryController">
+    <plugin filename="libgz-sim-joint-trajectory-controller-system.so" name="gz::sim::systems::JointTrajectoryController">
       <topic>/gazebo/joint_trajectory</topic>
     </plugin>
-    <plugin filename="gz-sim-joint-state-publisher-system" name="gz::sim::systems::JointStatePublisher">
+    <plugin filename="libgz-sim-joint-state-publisher-system.so" name="gz::sim::systems::JointStatePublisher">
       <topic>/gazebo/joint_states</topic>
       <joint_name>joint_1</joint_name>
